File: HW_LED_Large/HW_LED_Large.kicad_sch (KiCad schematic)
At the start: 81 parts

Commit message: Parts selected
Parts:
- added D41: D_Small, symbol Device:D_Small
- added H1, H2, H3, H4: MountingHole_Pad, MountingHole:MountingHole_4.3mm_M4_ISO7380_Pad, symbol Mechanical:MountingHole_Pad
- added J1: Barrel_Jack, Connector_BarrelJack:BarrelJack_CUI_PJ-063AH_Horizontal, symbol Connector:Barrel_Jack
Connections:
- net +5V: now also D41.1 (K)
- net D9: no longer D1.4 (DIN), D1.4 (DIN), D1.4 (DIN)
- net GND: now also H1.1, H2.1, H3.1, H4.1, J1.2
- net LED_CONT_1: now reaches D2.2 (DOUT)
- net LED_CONT_1: now also D1.4 (DIN)
- net LED_CONT_3: now reaches D2.2 (DOUT)
- net LED_CONT_3: now also D1.4 (DIN)
- net LED_CONT_2: now reaches D2.2 (DOUT)
- net LED_CONT_2: now also D1.4 (DIN)
- new net: D41.2 (A), J1.1
- no-connect marks 0 -> 1
Other:
- moved on the sheet: A1, C1, C2, D1, D2

Commit message: Added diode footprint
Parts:
- D41: footprint (none) -> Diode_SMD:D_SMA_Handsoldering
Changed lines of the file:
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@@
       (effects (font (size 1.27 1.27)))
     )
-    (property "Footprint" "" (at 250.19 20.32 90)
+    (property "Footprint" "Diode_SMD:D_SMA_Handsoldering" (at 250.19 20.32 90)
       (effects (font (size 1.27 1.27)) hide)
     )

Commit message: Added pins for ultrasonic sensor
Parts:
- added J2: Conn_01x04_Socket, Connector_PinSocket_2.54mm:PinSocket_1x04_P2.54mm_Vertical, symbol Connector:Conn_01x04_Socket
Connections:
- net +5V: now also J2.1 (Pin_1)
- net D5: now also J2.2 (Pin_2)
- net D6: now also J2.3 (Pin_3)
- net GND: now also J2.4 (Pin_4)
Other:
- note added: "2.54mm connector for the ultrasonic sensor"
Changed lines of the file:
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@@
     (stroke (width 0) (type default))
   )
+  (wire (pts (xy 247.65 77.47) (xy 247.65 80.01))
+    (stroke (width 0) (type default))
+  )
   (wire (pts (xy 40.64 26.67) (xy 40.64 27.94))
     (stroke (width 0) (type default))
@@
     (stroke (width 0) (type default))
   )
+  (wire (pts (xy 247.65 85.09) (xy 254 85.09))
+    (stroke (width 0) (type default))
+  )
   (wire (pts (xy 111.76 64.77) (xy 111.76 66.04))
     (stroke (width 0) (type default))
@@
     (stroke (width 0) (type default))
   )
+  (wire (pts (xy 247.65 87.63) (xy 254 87.63))
+    (stroke (width 0) (type default))
+  )
   (wire (pts (xy 186.69 36.83) (xy 189.23 36.83))
     (stroke (width 0) (type default))
@@
     (stroke (width 0) (type default))
   )
+  (wire (pts (xy 247.65 82.55) (xy 254 82.55))
+    (stroke (width 0) (type default))
+  )
   (wire (pts (xy 36.83 144.78) (xy 36.83 135.89))
     (stroke (width 0) (type default))
@@
     (stroke (width 0) (type default))
   )
+  (wire (pts (xy 247.65 88.9) (xy 247.65 87.63))
+    (stroke (width 0) (type default))
+  )
   (wire (pts (xy 36.83 96.52) (xy 40.64 96.52))
     (stroke (width 0) (type default))
@@
     (stroke (width 0) (type default))
   )
+  (wire (pts (xy 247.65 80.01) (xy 254 80.01))
+    (stroke (width 0) (type default))
+  )
   (wire (pts (xy 93.98 135.89) (xy 93.98 137.16))
     (stroke (width 0) (type default))
@@
     (stroke (width 0) (type default))
   )
+  (text "2.54mm connector for\nthe ultrasonic sensor" (at 260.35 80.01 0)
+    (effects (font (size 1.27 1.27)) (justify left bottom))
+  )
   (label "D12" (at 238.76 143.51 0) (fields_autoplaced)
     (effects (font (size 1.27 1.27)) (justify left bottom))
@@
     (effects (font (size 1.27 1.27)) (justify right bottom))
   )
+  (label "D5" (at 247.65 82.55 0) (fields_autoplaced)
+    (effects (font (size 1.27 1.27)) (justify left bottom))
+  )
   (label "A3" (at 279.4 135.89 180) (fields_autoplaced)
     (effects (font (size 1.27 1.27)) (justify right bottom))
@@
     (effects (font (size 1.27 1.27)) (justify right bottom))
   )
+  (label "D6" (at 247.65 85.09 0) (fields_autoplaced)
+    (effects (font (size 1.27 1.27)) (justify left bottom))
+  )
   (label "TX1" (at 238.76 115.57 0) (fields_autoplaced)
     (effects (font (size 1.27 1.27)) (justify left bottom))
@@
     )
   )
+  (symbol (lib_id "Connector:Conn_01x04_Socket") (at 259.08 82.55 0) (unit 1)
+    (in_bom yes) (on_board yes) (dnp no) (fields_autoplaced)
+    (property "Reference" "J2" (at 260.35 82.55 0)
+      (effects (font (size 1.27 1.27)) (justify left))
+    )
+    (property "Value" "Conn_01x04_Socket" (at 260.35 85.09 0)
+      (effects (font (size 1.27 1.27)) (justify left))
+    )
+    (property "Footprint" "Connector_PinSocket_2.54mm:PinSocket_1x04_P2.54mm_Vertical" (at 259.08 82.55 0)
+      (effects (font (size 1.27 1.27)) hide)
+    )
+    (property "Datasheet" "~" (at 259.08 82.55 0)
+      (effects (font (size 1.27 1.27)) hide)
+    )
+    (pin "1")
+    (pin "2")
+    (pin "3")
+    (pin "4")
+    (instances
+      (project "HW_LED_Large"
+        (path "/fc941b1f-6a6d-41f8-8c26-6162d29cf04e"
+          (reference "J2") (unit 1)
+        )
+      )
+    )
+  )
   (symbol (lib_id "Mechanical:MountingHole_Pad") (at 257.81 52.07 270) (unit 1)
     (in_bom yes) (on_board yes) (dnp no) (fields_autoplaced)
@@
     )
   )
+  (symbol (lib_id "power:GND") (at 247.65 88.9 0) (unit 1)
+    (in_bom yes) (on_board yes) (dnp no)
+    (property "Reference" "#PWR0116" (at 247.65 95.25 0)
+      (effects (font (size 1.27 1.27)) hide)
+    )
+    (property "Value" "GND" (at 250.19 91.44 0)
+      (effects (font (size 1.27 1.27)))
+    )
+    (property "Footprint" "" (at 247.65 88.9 0)
+      (effects (font (size 1.27 1.27)) hide)
+    )
+    (property "Datasheet" "" (at 247.65 88.9 0)
+      (effects (font (size 1.27 1.27)) hide)
+    )
+    (pin "1")
+    (instances
+      (project "ArduinoLearningBoard"
+        (path "/f026cf48-5183-40e4-8329-69bf8f917527"
+          (reference "#PWR0116") (unit 1)
+        )
+      )
+      (project "HW_LED_Large"
+        (path "/fc941b1f-6a6d-41f8-8c26-6162d29cf04e"
+          (reference "#PWR094") (unit 1)
+        )
+      )
+    )
+  )
   (symbol (lib_id "LED:WS2812B") (at 54.61 152.4 0) (unit 1)
     (in_bom yes) (on_board yes) (dnp no)
@@
         )
       )
+    )
+  )
+  (symbol (lib_id "power:+5V") (at 247.65 77.47 0) (unit 1)
+    (in_bom yes) (on_board yes) (dnp no)
+    (property "Reference" "#PWR0137" (at 247.65 81.28 0)
+      (effects (font (size 1.27 1.27)) hide)
+    )
+    (property "Value" "+5V" (at 248.92 73.66 0)
+      (effects (font (size 1.27 1.27)))
+    )
+    (property "Footprint" "" (at 247.65 77.47 0)
+      (effects (font (size 1.27 1.27)) hide)
+    )
+    (property "Datasheet" "" (at 247.65 77.47 0)
+      (effects (font (size 1.27 1.27)) hide)
+    )
+    (pin "1")
+    (instances
+      (project "ArduinoLearningBoard"
+        (path "/f026cf48-5183-40e4-8329-69bf8f917527"
+          (reference "#PWR0137") (unit 1)
+        )
+      )
+      (project "HW_LED_Large"
+        (path "/fc941b1f-6a6d-41f8-8c26-6162d29cf04e"
+          (reference "#PWR095") (unit 1)
+        )
+      )
